File: Hardware/Elektor_LoR_Node.sch (KiCad schematic (older format))
At the start: 62 parts, among them IC1 TLV809K33, IC2 TLV75533PDBV, IC3 AT25SF081-SSHD-X, IC4 STM32F072C8Tx, IC5 ATECC608A, IC6 MAX40200, IC7 MAX40200, K1 Conn_01x01_Female, K2 Conn_01x02_Male, K3 Conn_01x04_Male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

Commit message: Files for Version 3.2
Fixed library problems within the project
Parts:
- ANT1: value Antenna -> 868MHz; symbol LoRa_Tracker-rescue:Antenna-Device -> Device:Antenna
- BT1, BT2: symbol LoRa_Tracker-rescue:Battery_Cell-Device -> Device:Battery_Cell
- C1, C10, C11, C12, C17, C18, C2, C3, C5, C7, C8, C9: symbol LoRa_Tracker-rescue:C_Small-Device -> Device:C_Small
- C6: value 100nF -> 470nF; symbol LoRa_Tracker-rescue:C_Small-Device -> Device:C_Small
- D1: symbol LoRa_Tracker-rescue:1N4001-Diode -> Diode:1N4001
- F1, F2: symbol LoRa_Tracker-rescue:Fuse_Small-Device -> Device:Fuse_Small
- IC1: symbol LoRa_Tracker-rescue:TLV809K33-TLV803EA26DBZR -> TLV803EA26DBZR:TLV809K33
- IC3: symbol LoRa_Tracker-rescue:AT25SF081-SSHD-X-Memory_Flash -> Memory_Flash:AT25SF081-SSHD-X
- IC5: symbol LoRa_Tracker-rescue:ATECC608A-ATECC608A -> ATECC608A:ATECC608A
- K1: value Conn_01x01_Female -> (none)
- MOD1: value RFM95W-868S2 -> RFM95W
- R1, R4, R5, R6, R7, R8, R9: symbol LoRa_Tracker-rescue:R_Small-Device -> Device:R_Small
- S1, S2: symbol LoRa_Tracker-rescue:SW_Push-Switch -> Switch:SW_Push
- T1: symbol LoRa_Tracker-rescue:SI2347DS-SI2347DS -> SI2347DS:SI2347DS
- X1: symbol LoRa_Tracker-rescue:ASH7KW-Elektor_Abracon -> Elektor_Abracon:ASH7KW
Connections:
- net labels added: PA10, PA9, PB12, PB13, PB14, PB15
- net labels removed: UNUSED_00, UNUSED_01, UNUSED_02, UNUSED_03, UNUSED_04, UNUSED_05
- wire segments 283 -> 274
Other:
- note added: "Copyright Elektor 2019.\nThis documentation describes Open Hardware and is licensed under the CERN OHL v. 1.2.\nYou may redistribute and modify this documentation \nunder the terms of the CERN OHL v.1.2. (http://ohwr.org/cernohl). \nThis documentation is distributed \nWITHOUT ANY EXPRESS OR IMPLIED WARRANTY, INCLUDING OF MERCHANTABILITY,\nSATISFACTORY QUALITY AND FITNESS FOR A PARTICULAR PURPOSE.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"
- moved on the sheet: C13, C14, C16, C19, C20, C21, C4, H1, H2, IC6, JP1, K1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
